Commit message: changed urdf, visual is now working, collision is simplified for speed postprocessing setup is working

File: kuka_arm/urdf/kr210.urdf.xacro (robot description, xacro)
@@ -28,14 +28,14 @@
       <origin xyz="0 0 0" rpy="${-pi/2} 0 0"/>
       <geometry>
-        <mesh filename="package://kuka_arm/meshes/kr210l150/visual/base_link.dae"/>
-      </geometry>
-      <material name="">
-        <color rgba="0.75294 0.75294 0.75294 1"/>
-      </material>
-    </visual>
-    <collision>
-      <origin xyz="0 0 0" rpy="${-pi/2} 0 0"/>
-      <geometry>
         <mesh filename="package://kuka_arm/meshes/kr210l150/collision/base_link.stl"/>
+      </geometry>
+      <material name="">
+        <color rgba="0.75294 0.75294 0.75294 1"/>
+      </material>
+    </visual>
+    <collision>
+      <origin xyz="0 0 0.15" rpy="0 0 0"/>
+      <geometry>
+        <box size="1 1 0.3" />
       </geometry>
     </collision>
@@ -50,14 +50,14 @@
       <origin xyz="0 0 0" rpy="0 0 0"/>
       <geometry>
-        <mesh filename="package://kuka_arm/meshes/kr210l150/visual/link_1.dae"/>
-      </geometry>
-      <material name="">
-        <color rgba="0.75294 0.75294 0.75294 1"/>
-      </material>
-    </visual>
-    <collision>
-      <origin xyz="0 0 0" rpy="0 0 0"/>
-      <geometry>
         <mesh filename="package://kuka_arm/meshes/kr210l150/collision/link_1.stl"/>
+      </geometry>
+      <material name="">
+        <color rgba="0.75294 0.75294 0.75294 1"/>
+      </material>
+    </visual>
+    <collision>
+      <origin xyz="0 0 0.325" rpy="0 0 0"/>
+      <geometry>
+        <box size="1 1 0.65" />
       </geometry>
     </collision>
@@ -70,16 +70,16 @@
     </inertial>
     <visual>
-      <origin xyz="0 0 0" rpy="${-pi/2} 0 0"/>
-      <geometry>
-        <mesh filename="package://kuka_arm/meshes/kr210l150/visual/link_2.dae"/>
-      </geometry>
-      <material name="">
-        <color rgba="0.75294 0.75294 0.75294 1"/>
-      </material>
-    </visual>
-    <collision>
       <origin xyz="0 0 0" rpy="0 0 0"/>
       <geometry>
         <mesh filename="package://kuka_arm/meshes/kr210l150/collision/link_2.stl"/>
+      </geometry>
+      <material name="">
+        <color rgba="0.75294 0.75294 0.75294 1"/>
+      </material>
+    </visual>
+    <collision>
+      <origin xyz="0 -0.2 0.8" rpy="0 0 0"/>
+      <geometry>
+        <box size="0.4 0.4 1.6" />
       </geometry>
     </collision>
@@ -92,16 +92,16 @@
     </inertial>
     <visual>
-      <origin xyz="0 -0.184 0" rpy="${-pi/2} 0 0"/>
-      <geometry>
-        <mesh filename="package://kuka_arm/meshes/kr210l150/visual/link_3.dae"/>
-      </geometry>
-      <material name="">
-        <color rgba="0.75294 0.75294 0.75294 1"/>
-      </material>
-    </visual>
-    <collision>
       <origin xyz="0 -0.184 0" rpy="0 0 0"/>
       <geometry>
         <mesh filename="package://kuka_arm/meshes/kr210l150/collision/link_3.stl"/>
+      </geometry>
+      <material name="">
+        <color rgba="0.75294 0.75294 0.75294 1"/>
+      </material>
+    </visual>
+    <collision>
+      <origin xyz="0.2 0 0" rpy="0 0 0"/>
+      <geometry>
+        <box size="1.35 0.5 0.5" />
       </geometry>
     </collision>
@@ -114,16 +114,16 @@
     </inertial>
     <visual>
-      <origin xyz="0 0 0" rpy="${-pi/2} 0 0"/>
-      <geometry>
-        <mesh filename="package://kuka_arm/meshes/kr210l150/visual/link_4.dae"/>
-      </geometry>
-      <material name="">
-        <color rgba="0.75294 0.75294 0.75294 1"/>
-      </material>
-    </visual>
-    <collision>
       <origin xyz="0 0 0" rpy="0 0 0"/>
       <geometry>
         <mesh filename="package://kuka_arm/meshes/kr210l150/collision/link_4.stl"/>
+      </geometry>
+      <material name="">
+        <color rgba="0.75294 0.75294 0.75294 1"/>
+      </material>
+    </visual>
+    <collision>
+      <origin xyz="0.315 0 0" rpy="0 0 0"/>
+      <geometry>
+        <box size="0.63 0.35 0.25" />
       </geometry>
     </collision>
@@ -136,16 +136,16 @@
     </inertial>
     <visual>
-      <origin xyz="0 0 0" rpy="${-pi/2} 0 0"/>
-      <geometry>
-        <mesh filename="package://kuka_arm/meshes/kr210l150/visual/link_5.dae"/>
-      </geometry>
-      <material name="">
-        <color rgba="0.75294 0.75294 0.75294 1"/>
-      </material>
-    </visual>
-    <collision>
       <origin xyz="0 0 0" rpy="0 0 0"/>
       <geometry>
         <mesh filename="package://kuka_arm/meshes/kr210l150/collision/link_5.stl"/>
+      </geometry>
+      <material name="">
+        <color rgba="0.75294 0.75294 0.75294 1"/>
+      </material>
+    </visual>
+    <collision>
+      <origin xyz="0 0 0" rpy="0 0 0"/>
+      <geometry>
+        <box size="0.34 0.23 0.23" />
       </geometry>
     </collision>
@@ -160,5 +160,5 @@
       <origin xyz="0 0 0" rpy="0 0 0"/>
       <geometry>
-        <mesh filename="package://kuka_arm/meshes/kr210l150/visual/link_6.dae"/>
+        <mesh filename="package://kuka_arm/meshes/kr210l150/collision/link_6.stl"/>
       </geometry>
       <material name="">

Commit message: collision checking debuggable, seems to work in many cases, some false positives/wrong visualization planning with collision avoidance is not working

File: kuka_arm/urdf/kr210.urdf.xacro (robot description, xacro)
@@ -274,16 +274,4 @@
     <!-- kinect camera -->
     <link name="kinect_link">
-      <collision>
-        <origin xyz="0 0 0" rpy="0 0 0"/>
-        <geometry>
-      <box size="0.1 0.1 0.1"/>
-        </geometry>
-      </collision>
-      <visual>
-        <origin xyz="0 0 0" rpy="0 0 0"/>
-        <geometry>
-              <box size="0.1 0.1 0.1"/>
-        </geometry>
-      </visual>
       <inertial>
         <mass value="1e-5" />

Commit message: probably found a bug in stomps gradient cost function disabled octomap scan topic reenabled optimizing after valid trajectory, working raise max_distance, planer tries to plan as far away from obstacle as possible adjust camera4 position insertPointcloud now publishes all pointclouds maps generated raise voxel size to 10 cm in voxblox and move_group instance misuse updateMesh timer to publish pointclouds periodically

File: kuka_arm/urdf/kr210.urdf.xacro (robot description, xacro)
@@ -328,5 +328,5 @@
                <joint name="camera4_joint" type="fixed">
                   <axis xyz="0 1 0" />
-                  <origin xyz="1 0 5" rpy="0 1 0"/>
+                  <origin xyz="0 0 5" rpy="0 1.2 0"/>
                   <parent link="base_link"/>
                   <child link="camera4_link"/>
