Commit message: add depth camera to gazebo model

File: kuka_arm/urdf/kr210.gazebo.xacro (robot description, xacro)
@@ -82,3 +82,45 @@
     </plugin>
   </gazebo>
+  <gazebo reference="kinect_link">
+      <sensor type="depth" name="openni_camera_camera">
+          <always_on>1</always_on>
+          <visualize>true</visualize>
+          <camera>
+              <horizontal_fov>1.047</horizontal_fov>
+              <image>
+                  <width>100</width>
+                  <height>80</height>
+                  <format>R8G8B8</format>
+              </image>
+              <depth_camera>
+              </depth_camera>
+              <clip>
+                  <near>0.1</near>
+                  <far>10</far>
+              </clip>
+          </camera>
+          <plugin name="camera_controller" filename="libgazebo_ros_openni_kinect.so">
+              <alwaysOn>true</alwaysOn>
+                  <updateRate>10.0</updateRate>
+                  <cameraName>camera</cameraName>
+                  <frameName>kinect_link_optical_frame</frameName>
+              <imageTopicName>rgb/image_raw</imageTopicName>
+              <depthImageTopicName>depth/image_raw</depthImageTopicName>
+              <pointCloudTopicName>depth/points</pointCloudTopicName>
+              <cameraInfoTopicName>rgb/camera_info</cameraInfoTopicName>
+              <depthImageCameraInfoTopicName>depth/camera_info</depthImageCameraInfoTopicName>
+              <pointCloudCutoff>0.4</pointCloudCutoff>
+                  <hackBaseline>0.07</hackBaseline>
+                  <distortionK1>0.0</distortionK1>
+                  <distortionK2>0.0</distortionK2>
+                  <distortionK3>0.0</distortionK3>
+                  <distortionT1>0.0</distortionT1>
+                  <distortionT2>0.0</distortionT2>
+              <CxPrime>0.0</CxPrime>
+              <Cx>0.0</Cx>
+              <Cy>0.0</Cy>
+              <focalLength>0.0</focalLength>
+              </plugin>
+      </sensor>
+  </gazebo>
 </robot>

File: kuka_arm/urdf/kr210.urdf.xacro (robot description, xacro)
@@ -260,4 +260,36 @@
     </collision>
   </link>
+ <joint name="kinect_joint_optical_frame" type="fixed">
+      <origin xyz="0 0 0" rpy="-1.58 0 -1.58"/>
+      <parent link="kinect_link"/>
+      <child link="kinect_link_optical_frame"/>
+    </joint>
+    <link name="kinect_link_optical_frame"/>
+   <joint name="kinect_joint" type="fixed">
+      <axis xyz="0 1 0" />
+      <origin xyz="0 0 0.3" rpy="0 0 0"/>
+      <parent link="link_4"/>
+      <child link="kinect_link"/>
+    </joint>
+    <!-- kinect camera -->
+    <link name="kinect_link">
+      <collision>
+        <origin xyz="0 0 0" rpy="0 0 0"/>
+        <geometry>
+      <box size="0.1 0.1 0.1"/>
+        </geometry>
+      </collision>
+      <visual>
+        <origin xyz="0 0 0" rpy="0 0 0"/>
+        <geometry>
+              <box size="0.1 0.1 0.1"/>
+        </geometry>
+      </visual>
+      <inertial>
+        <mass value="1e-5" />
+        <origin xyz="0 0 0" rpy="0 0 0"/>
+        <inertia ixx="1e-6" ixy="0" ixz="0" iyy="1e-6" iyz="0" izz="1e-6" />
+      </inertial>
+    </link>
   <joint name="right_gripper_finger_joint" type="prismatic">
     <origin rpy="0 0 0" xyz="0.15 -0.0725 0" />

Commit message: added 3 more cameras to simulation

File: kuka_arm/urdf/kr210.gazebo.xacro (robot description, xacro)
@@ -90,6 +90,6 @@
               <horizontal_fov>1.2</horizontal_fov>
               <image>
-                  <width>100</width>
-                  <height>80</height>
+                  <width>50</width>
+                  <height>40</height>
                   <format>R8G8B8</format>
               </image>
@@ -125,3 +125,132 @@
       </sensor>
   </gazebo>
+    <gazebo reference="camera2_link">
+        <sensor type="depth" name="camera2">
+            <always_on>1</always_on>
+             <update_rate>30.0</update_rate>
+            <visualize>true</visualize>
+            <camera>
+                <horizontal_fov>2</horizontal_fov>
+                <image>
+                    <width>100</width>
+                    <height>50</height>
+                    <format>R8G8B8</format>
+                </image>
+                <depth_camera>
+                </depth_camera>
+                <clip>
+                    <near>0.1</near>
+                    <far>5</far>
+                </clip>
+            </camera>
+            <plugin name="camera2_controller" filename="libgazebo_ros_openni_kinect.so">
+                <alwaysOn>true</alwaysOn>
+                    <updateRate>30.0</updateRate>
+                    <cameraName>camera2</cameraName>
+                    <frameName>camera2_optical_frame</frameName>
+                <imageTopicName>rgb/image_raw</imageTopicName>
+                <depthImageTopicName>depth/image_raw</depthImageTopicName>
+                <pointCloudTopicName>depth/points</pointCloudTopicName>
+                <cameraInfoTopicName>rgb/camera_info</cameraInfoTopicName>
+                <depthImageCameraInfoTopicName>depth/camera_info</depthImageCameraInfoTopicName>
+                <pointCloudCutoff>0.4</pointCloudCutoff>
+                    <hackBaseline>0.07</hackBaseline>
+                    <distortionK1>0.0</distortionK1>
+                    <distortionK2>0.0</distortionK2>
+                    <distortionK3>0.0</distortionK3>
+                    <distortionT1>0.0</distortionT1>
+                    <distortionT2>0.0</distortionT2>
+                <CxPrime>0.0</CxPrime>
+                <Cx>0.0</Cx>
+                <Cy>0.0</Cy>
+                <focalLength>0.0</focalLength>
+                </plugin>
+        </sensor>
+    </gazebo>
+     <gazebo reference="camera3_link">
+            <sensor type="depth" name="camera3">
+                <always_on>1</always_on>
+                 <update_rate>30.0</update_rate>
+                <visualize>true</visualize>
+                <camera>
+                    <horizontal_fov>2</horizontal_fov>
+                    <image>
+                        <width>100</width>
+                        <height>50</height>
+                        <format>R8G8B8</format>
+                    </image>
+                    <depth_camera>
+                    </depth_camera>
+                    <clip>
+                        <near>0.1</near>
+                        <far>5</far>
+                    </clip>
+                </camera>
+                <plugin name="camera3_controller" filename="libgazebo_ros_openni_kinect.so">
+                    <alwaysOn>true</alwaysOn>
+                        <updateRate>30.0</updateRate>
+                        <cameraName>camera3</cameraName>
+                        <frameName>camera3_optical_frame</frameName>
+                    <imageTopicName>rgb/image_raw</imageTopicName>
+                    <depthImageTopicName>depth/image_raw</depthImageTopicName>
+                    <pointCloudTopicName>depth/points</pointCloudTopicName>
+                    <cameraInfoTopicName>rgb/camera_info</cameraInfoTopicName>
+                    <depthImageCameraInfoTopicName>depth/camera_info</depthImageCameraInfoTopicName>
+                    <pointCloudCutoff>0.4</pointCloudCutoff>
+                        <hackBaseline>0.07</hackBaseline>
+                        <distortionK1>0.0</distortionK1>
+                        <distortionK2>0.0</distortionK2>
+                        <distortionK3>0.0</distortionK3>
+                        <distortionT1>0.0</distortionT1>
+                        <distortionT2>0.0</distortionT2>
+                    <CxPrime>0.0</CxPrime>
+                    <Cx>0.0</Cx>
+                    <Cy>0.0</Cy>
+                    <focalLength>0.0</focalLength>
+                    </plugin>
+            </sensor>
+        </gazebo>
+             <gazebo reference="camera4_link">
+                    <sensor type="depth" name="camera4">
+                        <always_on>1</always_on>
+                         <update_rate>30.0</update_rate>
+                        <visualize>true</visualize>
+                        <camera>
+                            <horizontal_fov>1</horizontal_fov>
+                            <image>
+                                <width>100</width>
+                                <height>100</height>
+                                <format>R8G8B8</format>
+                            </image>
+                            <depth_camera>
+                            </depth_camera>
+                            <clip>
+                                <near>0.1</near>
+                                <far>6</far>
+                            </clip>
+                        </camera>
+                        <plugin name="camera4_controller" filename="libgazebo_ros_openni_kinect.so">
+                            <alwaysOn>true</alwaysOn>
+                                <updateRate>30.0</updateRate>
+                                <cameraName>camera4</cameraName>
+                                <frameName>camera4_optical_frame</frameName>
+                            <imageTopicName>rgb/image_raw</imageTopicName>
+                            <depthImageTopicName>depth/image_raw</depthImageTopicName>
+                            <pointCloudTopicName>depth/points</pointCloudTopicName>
+                            <cameraInfoTopicName>rgb/camera_info</cameraInfoTopicName>
+                            <depthImageCameraInfoTopicName>depth/camera_info</depthImageCameraInfoTopicName>
+                            <pointCloudCutoff>0.4</pointCloudCutoff>
+                                <hackBaseline>0.07</hackBaseline>
+                                <distortionK1>0.0</distortionK1>
+                                <distortionK2>0.0</distortionK2>
+                                <distortionK3>0.0</distortionK3>
+                                <distortionT1>0.0</distortionT1>
+                                <distortionT2>0.0</distortionT2>
+                            <CxPrime>0.0</CxPrime>
+                            <Cx>0.0</Cx>
+                            <Cy>0.0</Cy>
+                            <focalLength>0.0</focalLength>
+                            </plugin>
+                    </sensor>
+                </gazebo>
 </robot>

File: kuka_arm/urdf/kr210.urdf.xacro (robot description, xacro)
@@ -260,5 +260,5 @@
     </collision>
   </link>
- <joint name="kinect_joint_optical_frame" type="fixed">
+    <joint name="kinect_joint_optical_frame" type="fixed">
       <origin xyz="0 0 0" rpy="-1.58 0 -1.58"/>
       <parent link="kinect_link"/>
@@ -271,5 +271,5 @@
       <parent link="link_4"/>
       <child link="kinect_link"/>
-    </joint>
+   </joint>
     <!-- kinect camera -->
     <link name="kinect_link">
@@ -280,4 +280,64 @@
       </inertial>
     </link>
+    <joint name="camera2_optical_joint" type="fixed">
+      <origin xyz="0 0 0" rpy="-1.58 0 -1.58"/>
+      <parent link="camera2_link"/>
+      <child link="camera2_optical_frame"/>
+    </joint>
+    <link name="camera2_optical_frame"/>
+   <joint name="camera2_joint" type="fixed">
+      <axis xyz="0 1 0" />
+      <origin xyz="0 -3 2" rpy="0 0 1"/>
+      <parent link="base_link"/>
+      <child link="camera2_link"/>
+   </joint>
+    <!-- kinect camera -->
+    <link name="camera2_link">
+      <inertial>
+        <mass value="1e-5" />
+        <origin xyz="0 0 0" rpy="0 0 0"/>
+        <inertia ixx="1e-6" ixy="0" ixz="0" iyy="1e-6" iyz="0" izz="1e-6" />
+      </inertial>
+    </link>
+        <joint name="camera3_optical_joint" type="fixed">
+          <origin xyz="0 0 0" rpy="-1.58 0 -1.58"/>
+          <parent link="camera3_link"/>
+          <child link="camera3_optical_frame"/>
+        </joint>
+        <link name="camera3_optical_frame"/>
+       <joint name="camera3_joint" type="fixed">
+          <axis xyz="0 1 0" />
+          <origin xyz="0 3 2" rpy="0 0 -1"/>
+          <parent link="base_link"/>
+          <child link="camera3_link"/>
+       </joint>
+        <!-- kinect camera -->
+        <link name="camera3_link">
+          <inertial>
+            <mass value="1e-5" />
+            <origin xyz="0 0 0" rpy="0 0 0"/>
+            <inertia ixx="1e-6" ixy="0" ixz="0" iyy="1e-6" iyz="0" izz="1e-6" />
+          </inertial>
+        </link>
+                <joint name="camera4_optical_joint" type="fixed">
+                  <origin xyz="0 0 0" rpy="-1.58 0 -1.58"/>
+                  <parent link="camera4_link"/>
+                  <child link="camera4_optical_frame"/>
+                </joint>
+                <link name="camera4_optical_frame"/>
+               <joint name="camera4_joint" type="fixed">
+                  <axis xyz="0 1 0" />
+                  <origin xyz="1 0 5" rpy="0 1 0"/>
+                  <parent link="base_link"/>
+                  <child link="camera4_link"/>
+               </joint>
+                <!-- kinect camera -->
+                <link name="camera4_link">
+                  <inertial>
+                    <mass value="1e-5" />
+                    <origin xyz="0 0 0" rpy="0 0 0"/>
+                    <inertia ixx="1e-6" ixy="0" ixz="0" iyy="1e-6" iyz="0" izz="1e-6" />
+                  </inertial>
+                </link>
   <joint name="right_gripper_finger_joint" type="prismatic">
     <origin rpy="0 0 0" xyz="0.15 -0.0725 0" />

Commit message: untested changes

File: kuka_arm/urdf/kr210.gazebo.xacro (robot description, xacro)
@@ -217,5 +217,5 @@
                         <visualize>true</visualize>
                         <camera>
-                            <horizontal_fov>1</horizontal_fov>
+                            <horizontal_fov>1.2</horizontal_fov>
                             <image>
                                 <width>100</width>
@@ -227,5 +227,5 @@
                             <clip>
                                 <near>0.1</near>
-                                <far>6</far>
+                                <far>8</far>
                             </clip>
                         </camera>

File: kuka_arm/urdf/kr210.urdf.xacro (robot description, xacro)
@@ -328,5 +328,5 @@
                <joint name="camera4_joint" type="fixed">
                   <axis xyz="0 1 0" />
-                  <origin xyz="0 0 5" rpy="0 1.2 0"/>
+                  <origin xyz="-1 0 3.5" rpy="0 0.9 0"/>
                   <parent link="base_link"/>
                   <child link="camera4_link"/>

Commit message: make convert to octree optional make use freespace pointcloud optional move DistanceQuerry message in own package in order to build in one run lower self filter padding lower resolution of moving camera add option to insert esdf every n scans

File: kuka_arm/urdf/kr210.gazebo.xacro (robot description, xacro)
@@ -85,10 +85,10 @@
           <always_on>1</always_on>
            <update_rate>30.0</update_rate>
-          <visualize>true</visualize>
+          <visualize>false</visualize>
           <camera>
               <horizontal_fov>1.2</horizontal_fov>
               <image>
-                  <width>50</width>
-                  <height>40</height>
+                  <width>25</width>
+                  <height>20</height>
                   <format>R8G8B8</format>
               </image>
@@ -96,6 +96,6 @@
               </depth_camera>
               <clip>
-                  <near>0.1</near>
-                  <far>3</far>
+                  <near>0.01</near>
+                  <far>6</far>
               </clip>
           </camera>
@@ -110,6 +110,6 @@
               <cameraInfoTopicName>rgb/camera_info</cameraInfoTopicName>
               <depthImageCameraInfoTopicName>depth/camera_info</depthImageCameraInfoTopicName>
-              <pointCloudCutoff>0.4</pointCloudCutoff>
-                  <hackBaseline>0.07</hackBaseline>
+              <pointCloudCutoff>0.0</pointCloudCutoff>
+                  <hackBaseline>0.0</hackBaseline>
                   <distortionK1>0.0</distortionK1>
                   <distortionK2>0.0</distortionK2>

File: kuka_arm/urdf/kr210.urdf.xacro (robot description, xacro)
@@ -261,5 +261,5 @@
   </link>
     <joint name="kinect_joint_optical_frame" type="fixed">
-      <origin xyz="0 0 0" rpy="-1.58 0 -1.58"/>
+      <origin xyz="0 0 0" rpy="-1.57079632679 0 -1.57079632679"/>
       <parent link="kinect_link"/>
       <child link="kinect_link_optical_frame"/>
@@ -281,5 +281,5 @@
     </link>
     <joint name="camera2_optical_joint" type="fixed">
-      <origin xyz="0 0 0" rpy="-1.58 0 -1.58"/>
+      <origin xyz="0 0 0" rpy="-1.57079632679 0 -1.57079632679"/>
       <parent link="camera2_link"/>
       <child link="camera2_optical_frame"/>
@@ -301,5 +301,5 @@
     </link>
         <joint name="camera3_optical_joint" type="fixed">
-          <origin xyz="0 0 0" rpy="-1.58 0 -1.58"/>
+          <origin xyz="0 0 0" rpy="-1.57079632679 0 -1.57079632679"/>
           <parent link="camera3_link"/>
           <child link="camera3_optical_frame"/>
@@ -321,5 +321,5 @@
         </link>
                 <joint name="camera4_optical_joint" type="fixed">
-                  <origin xyz="0 0 0" rpy="-1.58 0 -1.58"/>
+                  <origin xyz="0 0 0" rpy="-1.57079632679 0 -1.57079632679"/>
                   <parent link="camera4_link"/>
                   <child link="camera4_optical_frame"/>
